Commit message: air urdf added

File: ethercat_diff_drive/description/config/motor_drive.urdf.xacro (robot description, xacro)
@@ -157,62 +157,4 @@
     <origin xyz="0 0 0.14" rpy="0 0 0"/>
   </joint>
-  <gazebo reference="lidar_link">
-    <sensor name="lidar" type="ray">
-      <always_on>true</always_on>
-      <visualize>true</visualize>
-      <update_rate>5</update_rate>
-      <ray>
-        <scan>
-          <horizontal>
-            <samples>360</samples>
-            <resolution>1.00000</resolution>
-            <min_angle>0.000000</min_angle>
-            <max_angle>6.280000</max_angle>
-          </horizontal>
-        </scan>
-        <range>
-          <min>0.120000</min>
-          <max>3.5</max>
-          <resolution>0.015000</resolution>
-        </range>
-        <noise>
-          <type>gaussian</type>
-          <mean>0.0</mean>
-          <stddev>0.01</stddev>
-        </noise>
-      </ray>
-      <plugin name="scan" filename="libgazebo_ros_ray_sensor.so">
-        <ros>
-          <remapping>~/out:=scan</remapping>
-        </ros>
-        <output_type>sensor_msgs/LaserScan</output_type>
-        <frame_name>lidar_link</frame_name>
-      </plugin>
-    </sensor>
-  </gazebo>
-  <gazebo>
-    <plugin name="object_controller" filename="libgazebo_ros_planar_move.so">
-        <ros>
-        <!-- Add a namespace -->
-          <!-- <namespace>/diff_drive_controller</namespace> -->
-          <!-- <remapping>cmd_vel:=diff_drive_controller/cmd_vel</remapping> -->
-          <!-- <remapping>odom:=diff_drive_controller/odom</remapping> -->
-        </ros>
-      <!-- Set control loop update rate -->
-      <update_rate>100</update_rate>
-      <!-- Set odom publish rate -->
-      <publish_rate>20</publish_rate>
-      <!-- Set if odom required -->
-      <publish_odom>false</publish_odom>
-      <publish_odom_tf>false</publish_odom_tf>
-      <!-- Frame IDs -->
-      <odometry_frame>odom</odometry_frame>
-      <robot_base_frame>base_link</robot_base_frame>
-      <!-- Set odom covariance -->
-      <covariance_x>0.0001</covariance_x>
-      <covariance_y>0.0001</covariance_y>
-      <covariance_yaw>0.01</covariance_yaw>
-    </plugin>
-  </gazebo>
   <xacro:include filename="$(find ethercat_diff_drive)/description/ros2_control/motor_diff_drive.ros2_control.xacro" />
   <xacro:motor_drive/>

File: ethercat_diff_drive/description/config/motor_drive_webots_urdf.xacro (robot description, xacro)
@@ -41,5 +41,5 @@
 </material>
 <!-- PROPERTIES -->
-<xacro:property name="base_laser_x" value="0.202"/>
+<xacro:property name="base_laser_x" value="0.272"/>
 <xacro:property name="base_laser_y" value="0.0"/>
 <xacro:property name="base_laser_z" value="-0.004"/>
@@ -243,5 +243,5 @@
       </collision>
     </link>
-    <joint name="caster_${side}_1_joint" type="fixed">
+    <joint name="caster_${side}_1_joint" type="continuous">
       <parent link="${parent}"/>
       <child link="caster_${side}_1_link"/>
@@ -249,9 +249,9 @@
       <axis xyz="0 0 1"/>
     </joint>
-    <joint name="caster_${side}_2_joint" type="fixed">
+    <joint name="caster_${side}_2_joint" type="continuous">
       <parent link="caster_${side}_1_link"/>
       <child link="caster_${side}_2_link"/>
       <origin xyz="-0.016 0.0000 -0.040" rpy="${-90.0 * deg_to_rad} 0 0"/>
-      <axis xyz="0 1 0"/>
+      <axis xyz="0 0 1"/>
     </joint>
   </xacro:macro>
@@ -292,5 +292,5 @@
           <ros>
               <enabled>true</enabled>
-              <updateRate>10</updateRate>
+              <updateRate>20</updateRate>
               <topicName>/scan</topicName>
               <alwaysOn>true</alwaysOn>
@@ -341,4 +341,28 @@
       </ec_module> -->
   </joint>
+  <joint name="caster_front_right_1_joint">
+    <state_interface name="position"/>
+  </joint>
+  <joint name="caster_front_left_1_joint">
+    <state_interface name="position"/>
+  </joint>
+  <joint name="caster_back_right_1_joint">
+    <state_interface name="position"/>
+  </joint>
+  <joint name="caster_back_left_1_joint">
+    <state_interface name="position"/>
+  </joint>
+  <joint name="caster_front_right_2_joint">
+    <state_interface name="position"/>
+  </joint>
+  <joint name="caster_front_left_2_joint">
+    <state_interface name="position"/>
+  </joint>
+  <joint name="caster_back_right_2_joint">
+    <state_interface name="position"/>
+  </joint>
+  <joint name="caster_back_left_2_joint">
+    <state_interface name="position"/>
+  </joint>
 </ros2_control>
 </robot>
