Commit message: sick mesh added

File: ethercat_diff_drive/description/config/air_urdf.xacro (robot description, xacro)
@@ -9,4 +9,7 @@
   <material name="white">
     <color rgba="1 1 1 1"/>
+  </material>
+  <material name="yellow">
+    <color rgba="1.0, 0.92, 0.016, 1.0"/>
   </material>
     <!-- Define some commonly used intertial properties  -->
@@ -244,9 +247,11 @@
     </collision>
     <visual>
-      <origin xyz="0 0 0" rpy="0 0 0"/>
-      <geometry>
-        <cylinder radius="0.0508" length="0.055"/>
-      </geometry>
-      <material name="lidar_visual">
+      <origin xyz="0 0 0" rpy="3.1415 0 0"/>
+      <geometry>
+        <!-- <cylinder radius="0.0508" length="0.055"/> -->
+        <mesh filename="package://ethercat_diff_drive/description/config/meshes/s300.obj" scale="0.001 0.001 0.001"/>
+      </geometry>
+        <material name="yellow"/>
+      <!-- <material name="lidar_visual">
         <color rgba="0.8 0 0 1"/>
         <ambient>0.0 0.0 0.0 1.0</ambient>
@@ -254,5 +259,5 @@
         <specular>0.0 0.0 0.0 1.0</specular>
         <emissive>0.0 0.0 0.0 1.0</emissive>
-      </material>
+      </material> -->
     </visual>
   </link>
@@ -260,5 +265,5 @@
     <parent link="base_link"/>
     <child link="laser_link_0"/>
-    <origin xyz="0.4 -0.28 0.18" rpy="0 0 -0.7854"/>
+    <origin xyz="0.4 -0.28 0.18" rpy="0 0 -2.356"/>
   </joint>
     <!-- ****************************** LASER 1 *****************************    -->
@@ -276,9 +281,11 @@
     </collision>
     <visual>
-      <origin xyz="0 0 0" rpy="0 0 0"/>
-      <geometry>
-        <cylinder radius="0.0508" length="0.055"/>
-      </geometry>
-      <material name="lidar_visual">
+      <origin xyz="0 0 0" rpy="3.1415 0 0"/>
+      <geometry>
+        <!-- <cylinder radius="0.0508" length="0.055"/> -->
+        <mesh filename="package://ethercat_diff_drive/description/config/meshes/s300.obj" scale="0.001 0.001 0.001"/>
+      </geometry>
+      <material name="yellow"/>
+      <!-- <material name="lidar_visual">
         <color rgba="0.8 0 0 1"/>
         <ambient>0.0 0.0 0.0 1.0</ambient>
@@ -286,5 +293,5 @@
         <specular>0.0 0.0 0.0 1.0</specular>
         <emissive>0.0 0.0 0.0 1.0</emissive>
-      </material>
+      </material> -->
     </visual>
   </link>
@@ -292,5 +299,5 @@
     <parent link="base_link"/>
     <child link="laser_link_1"/>
-    <origin xyz="-0.4 0.28 0.18" rpy="0 0 2.3562"/>
+    <origin xyz="-0.4 0.28 0.18" rpy="0 0 0.7854"/>
   </joint>
   <xacro:include filename="$(find ethercat_diff_drive)/description/ros2_control/motor_diff_drive.ros2_control.xacro" />

Commit message: urdf edit

File: ethercat_diff_drive/description/config/air_urdf.xacro (robot description, xacro)
@@ -11,5 +11,8 @@
   </material>
   <material name="yellow">
-    <color rgba="1.0, 0.92, 0.016, 1.0"/>
+    <color rgba="1.0 0.92 0.016 1"/>
+  </material>
+  <material name="grey">
+    <color rgba="0.7 0.7 0.7 1.0"/>
   </material>
     <!-- Define some commonly used intertial properties  -->
@@ -65,5 +68,5 @@
         <box size="${base_panel_length} ${base_width} ${base_tick}"/>
       </geometry>
-      <material name="white"/>
+       <material name="grey"/>
     </visual>
     <visual>
@@ -72,5 +75,5 @@
         <box size="${base_panel_length} ${base_width} ${base_tick}"/>
       </geometry>
-      <material name="white"/>
+       <material name="grey"/>
     </visual>
     <visual>
@@ -79,5 +82,5 @@
         <box size="${base_panel_length} ${base_panel_width} ${base_tick}"/>
       </geometry>
-      <material name="white"/>
+       <material name="grey"/>
     </visual>
     <visual>
@@ -86,5 +89,5 @@
         <box size="${base_panel_length} ${base_width} ${base_tick}"/>
       </geometry>
-      <material name="white"/>
+       <material name="grey"/>
     </visual>
     <visual>
@@ -93,5 +96,5 @@
         <box size="${base_panel_length} ${base_width} ${base_tick}"/>
       </geometry>
-      <material name="white"/>
+       <material name="grey"/>
     </visual>
     <collision>
@@ -113,5 +116,5 @@
     </visual>
       <collision>
-      <origin xyz="0.0 0.0 ${wheel_zoff+base_height+battery_height/2.0}" rpy="0 0 0"/>
+      <origin xyz="0.0 0.0 0.0" rpy="0 0 0"/>
       <geometry>
         <box size="${battery_length} ${battery_width} ${battery_height}"/>
@@ -166,5 +169,5 @@
       </geometry>
     </collision>
-    <xacro:sphere_inertia m="5" r="${(base_height/2+wheel_zoff)}"/>
+    <xacro:sphere_inertia m="0.5" r="${(base_height/2+wheel_zoff)}"/>
   </link>
   <joint name="front_left_caster_joint" type="fixed">
@@ -186,5 +189,5 @@
       </geometry>
     </collision>
-    <xacro:sphere_inertia m="5" r="${(base_height/2+wheel_zoff)}"/>
+    <xacro:sphere_inertia m="0.5" r="${(base_height/2+wheel_zoff)}"/>
   </link>
   <joint name="front_right_caster_joint" type="fixed">
@@ -206,5 +209,5 @@
       </geometry>
     </collision>
-    <xacro:sphere_inertia m="5" r="${(base_height/2+wheel_zoff)}"/>
+    <xacro:sphere_inertia m="0.5" r="${(base_height/2+wheel_zoff)}"/>
   </link>
   <joint name="rear_left_caster_joint" type="fixed">
@@ -226,5 +229,5 @@
       </geometry>
     </collision>
-    <xacro:sphere_inertia m="5" r="${(base_height/2+wheel_zoff)}"/>
+    <xacro:sphere_inertia m="0.5" r="${(base_height/2+wheel_zoff)}"/>
   </link>
   <joint name="rear_right_caster_joint" type="fixed">
@@ -243,9 +246,9 @@
       <origin xyz="0 0 0" rpy="0 0 0"/>
       <geometry>
-        <cylinder radius="0.0508" length="0.055"/>
-      </geometry>
-    </collision>
-    <visual>
-      <origin xyz="0 0 0" rpy="3.1415 0 0"/>
+        <cylinder radius="0.0508" length="0.18"/>
+      </geometry>
+    </collision>
+    <visual>
+      <origin xyz="0 0 0" rpy="3.1415 0 -1.5708"/>
       <geometry>
         <!-- <cylinder radius="0.0508" length="0.055"/> -->
@@ -265,5 +268,5 @@
     <parent link="base_link"/>
     <child link="laser_link_0"/>
-    <origin xyz="0.4 -0.28 0.18" rpy="0 0 -2.356"/>
+    <origin xyz="0.4 -0.28 0.18" rpy="0 0 -0.7854"/>
   </joint>
     <!-- ****************************** LASER 1 *****************************    -->
@@ -277,9 +280,9 @@
       <origin xyz="0 0 0" rpy="0 0 0"/>
       <geometry>
-        <cylinder radius="0.0508" length="0.055"/>
-      </geometry>
-    </collision>
-    <visual>
-      <origin xyz="0 0 0" rpy="3.1415 0 0"/>
+        <cylinder radius="0.0508" length="0.18"/>
+      </geometry>
+    </collision>
+    <visual>
+      <origin xyz="0 0 0" rpy="3.1415 0 -1.5708"/>
       <geometry>
         <!-- <cylinder radius="0.0508" length="0.055"/> -->
@@ -299,5 +302,5 @@
     <parent link="base_link"/>
     <child link="laser_link_1"/>
-    <origin xyz="-0.4 0.28 0.18" rpy="0 0 0.7854"/>
+    <origin xyz="-0.4 0.28 0.18" rpy="0 0 2.3562"/>
   </joint>
   <xacro:include filename="$(find ethercat_diff_drive)/description/ros2_control/motor_diff_drive.ros2_control.xacro" />

Commit message: urdf edit

File: ethercat_diff_drive/description/config/air_urdf.xacro (robot description, xacro)
@@ -61,5 +61,5 @@
         <box size="${base_panel_length} ${base_panel_width} ${base_tick}"/>
       </geometry>
-      <material name="white"/>
+      <material name="grey"/>
     </visual>
     <visual>
