Commit message: epos4 + gpio and beckhoff servo drive added

File: ethercat_diff_drive/description/config/air_urdf_el7221.xacro (robot description, xacro)
@@ -132,5 +132,5 @@
     <link name="joint_link_${prefix}">
       <visual>
-        <origin xyz="0 0 0" rpy="${pi/2} 0 0"/>
+        <origin xyz="0 0 0" rpy="0 0 0"/>
         <geometry>
           <cylinder radius="${wheel_radius}" length="${wheel_width}"/>
@@ -139,5 +139,5 @@
       </visual>
       <collision>
-        <origin xyz="0 0 0" rpy="${pi/2} 0 0"/>
+        <origin xyz="0 0 0" rpy="0 0 0"/>
         <geometry>
           <cylinder radius="${wheel_radius}" length="${wheel_width}"/>
@@ -149,6 +149,6 @@
       <parent link="base_link"/>
       <child link="joint_link_${prefix}"/>
-      <origin xyz="${x_reflect*wheel_xoff} ${y_reflect*(base_width/2+wheel_ygap)} ${wheel_radius}" rpy="0 0 0"/>
-      <axis xyz="0 1 0"/>
+      <origin xyz="${x_reflect*wheel_xoff} ${y_reflect*(base_width/2+wheel_ygap)} ${wheel_radius}" rpy="${y_reflect*pi/2} 0 0"/>
+      <axis xyz="0 0 1"/>
       <dynamics damping="10" friction="5"/>
     </joint>

File: ethercat_diff_drive/description/ros2_control/motor_diff_drive.ros2_control.xacro (robot description, xacro)
@@ -32,4 +32,20 @@
         </ec_module>
       </gpio>
+        <gpio name="gpio1">
+        <state_interface name="di.1"/>
+        <state_interface name="di.3"/>
+        <state_interface name="di.4"/>
+        <state_interface name="di.2"/>
+        <state_interface name="di.9"/>
+        <state_interface name="di.10"/>
+        <state_interface name="di.11"/>
+        <state_interface name="di.12"/>
+        <ec_module name="EL1809">
+          <plugin>ethercat_generic_plugins/GenericEcSlave</plugin>
+          <param name="alias">0</param>
+          <param name="position">5</param>
+          <param name="slave_config">$(find ethercat_diff_drive)/config/beckhoff_el1809.yaml</param>
+        </ec_module>
+      </gpio>
       <joint name="joint_1">
         <state_interface name="position"/>

File: ethercat_diff_drive/description/ros2_control/motor_drive_el7221.xacro (robot description, xacro)
@@ -6,5 +6,5 @@
         <plugin>ethercat_driver/EthercatDriver</plugin>
         <param name="master_id">0</param>
-        <param name="control_frequency">100</param>
+        <param name="control_frequency">500</param>
       </hardware>
       <gpio name="gpio0">
@@ -28,5 +28,5 @@
           <plugin>ethercat_generic_plugins/GenericEcSlave</plugin>
           <param name="alias">0</param>
-          <param name="position">6</param>
+          <param name="position">4</param>
           <param name="slave_config">$(find ethercat_diff_drive)/config/beckhoff_el2809.yaml</param>
         </ec_module>
@@ -34,8 +34,8 @@
       <gpio name="gpio1">
         <state_interface name="di.1"/>
-        <state_interface name="di.2"/>
         <state_interface name="di.3"/>
         <state_interface name="di.4"/>
-        <state_interface name="di.9"/>
+       <state_interface name="di.2"/>
+         <state_interface name="di.9"/>
         <state_interface name="di.10"/>
         <state_interface name="di.11"/>
@@ -44,5 +44,5 @@
           <plugin>ethercat_generic_plugins/GenericEcSlave</plugin>
           <param name="alias">0</param>
-          <param name="position">5</param>
+          <param name="position">3</param>
           <param name="slave_config">$(find ethercat_diff_drive)/config/beckhoff_el1809.yaml</param>
         </ec_module>
@@ -53,10 +53,10 @@
         <!-- <state_interface name="effort"/> -->
         <command_interface name="velocity"/>
-        <!-- <command_interface name="reset_fault"/> -->
+        <command_interface name="reset_fault"/>
         <ec_module name="Beckhoff">
           <plugin>ethercat_generic_plugins/EcCiA402Drive</plugin>
           <param name="alias">0</param>
-          <param name="position">3</param>
-          <!-- <param name="mode_of_operation">9</param> -->
+          <param name="position">1</param>
+          <param name="mode_of_operation">9</param>
           <param name="slave_config">$(find ethercat_diff_drive)/config/beckhoff_el7221-9015_slave_config.yaml</param>
         </ec_module>
@@ -67,10 +67,10 @@
         <!-- <state_interface name="effort"/> -->
         <command_interface name="velocity"/>
-        <!-- <command_interface name="reset_fault"/> -->
+        <command_interface name="reset_fault"/>
         <ec_module name="Beckhoff">
           <plugin>ethercat_generic_plugins/EcCiA402Drive</plugin>
           <param name="alias">0</param>
-          <param name="position">4</param>
-          <!-- <param name="mode_of_operation">9</param> -->
+          <param name="position">2</param>
+          <param name="mode_of_operation">9</param>
           <param name="slave_config">$(find ethercat_diff_drive)/config/beckhoff_el7221-9015_slave_config.yaml</param>
         </ec_module>

Commit message: added air_bringup with rtabmap slam

File: ethercat_diff_drive/description/config/air_urdf_el7221.xacro (robot description, xacro)
@@ -304,4 +304,27 @@
     <origin xyz="-0.4 0.28 0.18" rpy="0 0 2.3562"/>
   </joint>
+  <!-- RealSense D435i Camera -->
+  <link name="camera_link">
+    <visual>
+      <geometry>
+        <box size="0.025 0.09 0.025"/> <!-- Temsili kutu -->
+      </geometry>
+      <origin xyz="0 0 0" rpy="0 0 0"/>
+      <material name="black">
+        <color rgba="0 0 0 1"/>
+      </material>
+    </visual>
+    <inertial>
+      <mass value="0.1"/>
+      <inertia ixx="0.0001" ixy="0.0" ixz="0.0"
+               iyy="0.0001" iyz="0.0"
+               izz="0.0001"/>
+    </inertial>
+  </link>
+  <joint name="camera_joint" type="fixed">
+    <parent link="base_link"/>
+    <child link="camera_link"/>
+    <origin xyz="0.25 0.0 0.50" rpy="0 0 0"/>
+  </joint>
   <xacro:include filename="$(find ethercat_diff_drive)/description/ros2_control/motor_drive_el7221.xacro" />
   <xacro:motor_drive/>

File: ethercat_diff_drive/description/ros2_control/motor_drive_el7221.xacro (robot description, xacro)
@@ -17,5 +17,5 @@
         <command_interface name="do.11"/>
         <command_interface name="do.12"/>
-        <state_interface name="do.1"/>
+        <!-- <state_interface name="do.1"/>
         <state_interface name="do.2"/>
         <state_interface name="do.3"/>
@@ -24,5 +24,5 @@
         <state_interface name="do.10"/>
         <state_interface name="do.11"/>
-        <state_interface name="do.12"/>
+        <state_interface name="do.12"/> -->
         <ec_module name="EL2809">
           <plugin>ethercat_generic_plugins/GenericEcSlave</plugin>
@@ -36,6 +36,6 @@
         <state_interface name="di.3"/>
         <state_interface name="di.4"/>
-       <state_interface name="di.2"/>
-         <state_interface name="di.9"/>
+        <state_interface name="di.2"/>
+        <state_interface name="di.9"/>
         <state_interface name="di.10"/>
         <state_interface name="di.11"/>

Commit message: diff_drive_controller feedback velocity and rtmap db delete option

File: ethercat_diff_drive/description/config/air_urdf_el7221.xacro (robot description, xacro)
@@ -325,5 +325,5 @@
     <parent link="base_link"/>
     <child link="camera_link"/>
-    <origin xyz="0.25 0.0 0.50" rpy="0 0 0"/>
+    <origin xyz="0.29 0.04 0.46" rpy="0 0 0"/>
   </joint>
   <xacro:include filename="$(find ethercat_diff_drive)/description/ros2_control/motor_drive_el7221.xacro" />

File: ethercat_diff_drive/description/ros2_control/motor_drive_el7221.xacro (robot description, xacro)
@@ -50,5 +50,5 @@
       <joint name="joint_1">
         <state_interface name="position"/>
-        <!-- <state_interface name="velocity"/> -->
+        <state_interface name="velocity"/>
         <!-- <state_interface name="effort"/> -->
         <command_interface name="velocity"/>
@@ -64,5 +64,5 @@
       <joint name="joint_2">
         <state_interface name="position"/>
-        <!-- <state_interface name="velocity"/> -->
+        <state_interface name="velocity"/>
         <!-- <state_interface name="effort"/> -->
         <command_interface name="velocity"/>
